Commit message: Add URDF and Xacro files for robot components including common properties, mobile base, lidar, and Gazebo integration

File: ros_ws/src/my_robot_description/urdf/my_robot.urdf.xacro (robot description, xacro)
@@ -3,90 +3,7 @@
 <!--Bernardo Serravalle Resende-->
 <robot name="my_robot" xmlns:xacro="http://www.ros.org/wiki/xacro">
-    <xacro:property name="base_length" value="0.6" />
-    <xacro:property name="base_width" value="0.4" />
-    <xacro:property name="base_height" value="0.2" />
-    <xacro:property name="wheel_radius" value="0.1" />
-    <xacro:property name="wheel_length" value="0.05" />
-    <material name="gray">
-        <color rgba="0.7 0.7 0.7 1"/>
-    </material>
-    <material name="green">
-        <color rgba="0 0.6 0 1"/>
-    </material>
-    <material name="white">
-        <color rgba="1 1 1 1"/>
-    </material>
-    <link name="base_footprint"/>
-    <link name="base_link">
-        <visual>
-            <geometry>
-                <box size="${base_length} ${base_width} ${base_height}"/>
-            </geometry>
-            <origin xyz="0 0 ${base_height/2}" rpy="0 0 0"/>
-            <material name="green"/>
-        </visual>
-    </link>
-    <link name="lidar">
-        <visual>
-            <geometry>
-                <cylinder radius="0.1" length="0.05"/>
-            </geometry>
-            <origin xyz="0 0 0" rpy="0 0 0"/>
-            <material name="white"/>
-        </visual>
-    </link>
-    <link name="left_wheel_link">
-        <visual>
-            <geometry>
-                <cylinder radius="${wheel_radius}" length="${wheel_length}"/>
-            </geometry>
-            <origin xyz="0 0 0" rpy="${pi / 2} 0 0"/>
-            <material name="gray"/>
-        </visual>
-    </link>
-    <link name="right_wheel_link">
-        <visual>
-            <geometry>
-                <cylinder radius="${wheel_radius}" length="${wheel_length}"/>
-            </geometry>
-            <origin xyz="0 0 0" rpy="${pi / 2} 0 0"/>
-            <material name="gray"/>
-        </visual>
-    </link>
-    <link name="caster_wheel_link">
-        <visual>
-            <geometry>
-                <sphere radius="${wheel_radius / 2}"/>
-            </geometry>
-            <origin xyz="0 0 0" rpy="0 0 0"/>
-            <material name="gray"/>
-        </visual>
-    </link>
-    <joint name="base_joint" type="fixed">
-        <parent link="base_footprint"/>
-        <child link="base_link"/>
-        <origin xyz="0 0 ${wheel_radius}" rpy="0 0 0"/>
-    </joint>
-    <joint name="base_lidar_joint" type="fixed">
-        <parent link="base_link"/>
-        <child link="lidar"/>
-        <origin xyz="0 0 0.225" rpy="0 0 0"/>
-    </joint>
-    <joint name="base_left_wheel_joint" type="continuous">
-        <parent link="base_link"/>
-        <child link="left_wheel_link"/>
-        <origin xyz="${-base_length / 4.0} ${(base_width + wheel_length) / 2.0} 0" rpy="0 0 0"/>
-        <axis xyz="0 1 0"/>
-    </joint>
-    <joint name="base_right_wheel_joint" type="continuous">
-        <parent link="base_link"/>
-        <child link="right_wheel_link"/>
-        <origin xyz="${-base_length / 4.0} ${-(base_width + wheel_length) / 2.0} 0" rpy="0 0 0"/>
-        <axis xyz="0 1 0"/>
-    </joint>
-    <joint name="base_caster_wheel_joint" type="fixed">
-        <parent link="base_link"/>
-        <child link="caster_wheel_link"/>
-        <origin xyz="${base_length / 3.0} 0 ${-wheel_radius / 2.0}" rpy="0 0 0"/>
-    </joint>
+    <xacro:include filename="common_properties.xacro" />
+    <xacro:include filename="mobile_base.xacro" />
+    <xacro:include filename="mobile_base_gazebo.xacro" />
+    <xacro:include filename="lidar.xacro" />
 </robot>
